Commit message: bugfix: drive every robot in every simulator

File: arena_robots/components/camera/d435_depth/d435_depth.urdf.xacro (robot description, xacro)
@@ -12,7 +12,7 @@
       <origin xyz="0 0 0" rpy="0 0 0" />
     </xacro:sensor_d435>
-    <gazebo reference="${name}_link">
+    <gazebo reference="${name}_depth_frame">
       <sensor name="${name}" type="depth_camera">
-        <gz_frame_id>$(arg sim_path)/${name}_link</gz_frame_id>
+        <gz_frame_id>$(arg sim_path)/${name}_depth_frame</gz_frame_id>
         <always_on>1</always_on>
         <update_rate>30</update_rate>

File: arena_robots/components/camera/oakd_rgbd/oakd_rgb.urdf.xacro (robot description, xacro)
@@ -98,5 +98,5 @@
       <origin xyz="0 0 0" rpy="-${M_PI/2} 0 -${M_PI/2}" />
   </joint>
-  <gazebo reference="${name}_imu_joint">
+  <gazebo reference="${name}_imu_frame">
     <sensor name="${name}_imu" type="imu">
       <plugin filename="libgz-sim-imu-system" name="gz::sim::systems::Imu">

File: arena_robots/components/lidar/sick_microscan3/sick_microscan3.urdf.xacro (robot description, xacro)
@@ -12,5 +12,7 @@
                        node_namespace:=${None}
                        topic_prefix:=~/
-                       gpu:=false">
+                       gpu:=false
+                       half_angle:=2.39982772
+                       samples:=2751">
     <!-- node_namespace is used from node_name if not set -->
     <xacro:if value="${node_namespace == None}">
@@ -55,10 +57,10 @@
       min_range="0.05"
       max_range="64.0"
-      min_angle="-2.39982772"
-      max_angle="2.39982772"
+      min_angle="${-half_angle}"
+      max_angle="${half_angle}"
       frame_link="${frame_prefix}link"
       rate="33"
       resolution="0.00575"
-      samples="2751"
+      samples="${samples}"
     >
     </xacro:lidar_2d_plugin>

File: arena_robots/robots/a1/urdf/include/depthcamera.xacro (robot description, xacro)
@@ -25,7 +25,7 @@
       <origin xyz="0 0 0" rpy="${-pi/2} 0 ${-pi/2}"/>
       <parent link="${prefix}camera_${name}"/>
-      <child link="${prefix}camera_optical_${name}"/>
+      <child link="${prefix}camera_${name}_optical_frame"/>
     </joint>
-    <link name="${prefix}camera_optical_${name}"/>
+    <link name="${prefix}camera_${name}_optical_frame"/>
     <xacro:gz_rgbd_camera frame="${prefix}camera_${name}" sensor_name="${prefix}camera_${name}"
                           fov="2.094" width="640" height="480" near="0.05" far="8.0"

File: arena_robots/robots/go1/urdf/include/const.xacro (robot description, xacro)
@@ -41,6 +41,6 @@
     <xacro:property name="calf_max" value="-48"/>
     <xacro:property name="calf_min" value="-156"/>
-    <xacro:property name="calf_velocity_max" value="30.1"/>
-    <xacro:property name="calf_torque_max" value="23.7"/>
+    <xacro:property name="calf_velocity_max" value="20.06"/>
+    <xacro:property name="calf_torque_max" value="35.55"/>
     <!-- dynamics inertial value        total 12.84kg -->
     <!-- trunk -->

File: arena_robots/robots/go1/urdf/include/depthcamera.xacro (robot description, xacro)
@@ -34,10 +34,10 @@
       <origin xyz="0 0 0" rpy="${-pi/2} 0 ${-pi/2}"/>
       <parent link="${prefix}camera_${name}"/>
-      <child link="${prefix}camera_optical_${name}"/>
+      <child link="${prefix}camera_${name}_optical_frame"/>
     </joint>
-    <link name="${prefix}camera_optical_${name}"/>
+    <link name="${prefix}camera_${name}_optical_frame"/>
     <xacro:gz_rgbd_camera frame="${prefix}camera_${name}" sensor_name="${prefix}camera_${name}"
                           fov="2.094" width="928" height="800" near="0.1" far="5.0"
-                          update_rate="16" pose="0.04 0 0 0 0 0"/>
+                          update_rate="16"/>
   </xacro:macro>
 </robot>

File: arena_robots/robots/rbvogui/urdf/bodies/rbvogui/rbvogui_body.urdf.xacro (robot description, xacro)
@@ -14,5 +14,11 @@
     </joint>
     <!-- BASE_LINK -->
-    <link name="${prefix}base_link"/>
+    <link name="${prefix}base_link">
+      <inertial>
+        <mass value="25.0" />
+        <origin xyz="-0.012 0 0.2775" />
+        <xacro:solid_cuboid_inertia w="1.265" h="0.812" d="0.22" m="25.0"/>
+      </inertial>
+    </link>
     <!-- Chassis -->
     <joint name="${prefix}chassis_joint" type="fixed">
@@ -23,9 +29,4 @@
     <!-- Chassis -->
     <link name="${prefix}chassis_link">
-      <inertial>
-        <mass value="25.0" />
-        <origin xyz="0 0 0.10" />
-        <xacro:solid_cuboid_inertia w="1.265" h="0.812" d="0.22" m="25.0"/>
-      </inertial>
       <visual>
         <origin xyz="0 0 0" rpy="0 0 0" />

File: arena_robots/tests/golden/a1_default.urdf (robot description, URDF)
Before this commit: robot a1, 26 links, 25 joints
Links:
- removed link camera_optical_face
- added link camera_face_optical_frame
Joints:
- joint camera_optical_joint_face: child camera_optical_face -> camera_face_optical_frame

File: arena_robots/tests/golden/go1_default.urdf (robot description, URDF)
Before this commit: robot go1, 26 links, 25 joints
Links:
- removed link camera_optical_face
- added link camera_face_optical_frame
Joints:
- joint FL_calf_joint: limit lower=-2.722713633111154 upper=-0.8377580409572781 effort=23.7 velocity=30.1 -> lower=-2.722713633111154 upper=-0.8377580409572781 effort=35.55 velocity=20.06
- joint FR_calf_joint: limit lower=-2.722713633111154 upper=-0.8377580409572781 effort=23.7 velocity=30.1 -> lower=-2.722713633111154 upper=-0.8377580409572781 effort=35.55 velocity=20.06
- joint RL_calf_joint: limit lower=-2.722713633111154 upper=-0.8377580409572781 effort=23.7 velocity=30.1 -> lower=-2.722713633111154 upper=-0.8377580409572781 effort=35.55 velocity=20.06
- joint RR_calf_joint: limit lower=-2.722713633111154 upper=-0.8377580409572781 effort=23.7 velocity=30.1 -> lower=-2.722713633111154 upper=-0.8377580409572781 effort=35.55 velocity=20.06
- joint camera_optical_joint_face: child camera_optical_face -> camera_face_optical_frame

File: arena_robots/tests/golden/rbvogui_default.urdf (robot description, URDF)
Before this commit: robot rbvogui, 41 links, 40 joints
Links:
- link robot_base_link: mass None -> 25.0
- link robot_chassis_link: mass 25.0 -> None
