Commit message: bugfix: seat the go1 and a1 lidar on the trunk

File: arena_robots/tests/golden/a1_default.urdf (robot description, URDF)
Before this commit: robot a1, 26 links, 25 joints
Joints:
- joint lidar_joint: origin xyz=0 0 0.10 rpy=0 0 0 -> xyz=0 0 0.083 rpy=0 0 0

File: arena_robots/tests/golden/go1_default.urdf (robot description, URDF)
Before this commit: robot go1, 26 links, 25 joints
Joints:
- joint lidar_joint: origin xyz=0 0 0.10 rpy=0 0 0 -> xyz=0 0 0.096 rpy=0 0 0
